Commit message: Fix configuration and update README

File: description/lidar.xacro (robot description, xacro)
@@ -6,5 +6,5 @@
         <parent link="base_link"/>
         <child link="laser"/>
-        <origin xyz="0 0 0.2" rpy="0 0 0"/>
+        <origin xyz="0 0 0.2" rpy="0 0 ${pi}"/>
     </joint>
     <link name="laser">
